File: V3.1/eNode_Spark.brd (EAGLE design)
At the start: 30 x 65 mm, 65 parts, among them U1 USD-SOCKETSMD, U10 WM-N-BM-09, U2 BMP180, U3 HTU21DSMD, U6 MCP73831T-2ACI/OT, U7 TMP006, U8 OPA344, U9 ADMP401, X1 USB-MICROB

Commit message: Major commit
Updated rev from 3.0 to 3.1
Parts:
- removed D1: DIODE, Spark:DIODE-DO-220AA(SMP)
- removed SV1: (no value), con-lstb:MA04-1
- removed U$7: R8008-33, Spark:SOT23-5
- added C26: 0.1uF, rc-master-smd:C0402
- added CAM: (no value), Camera Header:MA04-1
- added JTAG: JTAG_CONNECTOR, JTAG Connector:JTAG_DIP
- added R17: 10K, rc-master-smd:R0402
- added R18: 1M, rc-master-smd:R0402
- added S3: MODE, TACT BUTTON:DTSM-3
- added S4: RESET, TACT BUTTON:DTSM-3
- added U5: HTU21DSMD, HTU21D:HTU21D
- C1, C3: value 4.7uF -> 10uF
- C10, C7: value 0.1uF -> 4.7uF
- C11: value 0.8pF +/-0.25pF (RF) -> 22uF; device Spark:C0402_B -> rc-master-smd:C0603
- C16: value 10nF -> 0.1uF
- C17: device Spark:C0402_B -> rc-master-smd:C0402
- C18: value 0.1uF -> 10nF; device Spark:C0402_B -> rc-master-smd:C0402
- C19: value 0.1uF -> 10uF; device Spark:C0402_B -> rc-master-smd:C1206/T
- C2: value 4.7uF -> 0.1uF
- C20, C21, C22: value 10uF -> 0.1uF; device Spark:C0402_B -> rc-master-smd:C0402
- C23: value 22uF -> 4.7uF; device rcl:C0603 -> rc-master-smd:C0402
- C24: value 22uF -> 1uF; device rcl:C0603 -> rc-master-smd:C0402
- C25: value 0.1uF -> 12pF; device adafruit:C0402 -> rc-master-smd:C0402
- C4: value 100pF -> 0.1uF
- C5: value 1uF -> 10uF
- C8: value 0.1uF -> 22uF; device rc-master-smd:C0402 -> rc-master-smd:C0603
- C9: value 10uF -> 0.8pF +/-0.25pF (RF); device rc-master-smd:C1206/T -> rc-master-smd:C0402
- L1: device Spark:L0402_B -> rc-master-smd:L0402
- LED1: value CREE_CLVBA-FKA -> (none)
- R1: value 100 -> 2K
- R10: device Spark:R0402_B -> rc-master-smd:R0402
- R11: value 4.7K -> 1K; device rc-master-smd:R0603 -> rc-master-smd:R0402
- R13: device rc-master-smd:R0603 -> rc-master-smd:R0402
- R14: value 1K -> 2.2K; device Spark:R0402_B -> rc-master-smd:R0402
- R15: value 1K -> 10K; device Spark:R0402_B -> rc-master-smd:R0402
- R16: value 4.7K -> 10K; device rc-master-smd:R0603 -> rc-master-smd:R0402
- R2: value 2K -> 100K; device rc-master-smd:R0603 -> rc-master-smd:R0402
- R3: value 22 -> 100; device Spark:R0402_B -> rc-master-smd:R0603
- R4: value 1.5K -> 22
- R5: value 100K -> 22
- R6, R7: value 10K -> 4.7K; device rc-master-smd:R0402 -> rc-master-smd:R0603
- R8: value 22 -> 10K; device Spark:R0402_B -> rc-master-smd:R0603
- R9: value 100K -> 1K; device Spark:R0402_B -> rc-master-smd:R0402
- S1, S2: device TACT BUTTON:TACTILE_SWITCH_SMD -> TACT BUTTON:TACTILE_SWITCH_SMD_LARGE_4
- U1: value USD-SOCKETSMD -> WM-N-BM-09; device MicroSD:MICRO-SD-SOCKET-PP -> Spark:WM-N-BM-09
- U10: value WM-N-BM-09 -> OPA344; device Spark:WM-N-BM-09 -> OPA344:SOT23-5
- U2: value BMP180 -> MCP73831T-2ACI/OT; device BMP180:BMP180 -> MCP73831T (LiPo Charger):SOT95P280X145-5N
- U3: value HTU21DSMD -> R8008-33; device HTU21D:HTU21D -> Spark:SOT23-5
- U6: value MCP73831T-2ACI/OT -> TMP006; device MCP73831T (LiPo Charger):SOT95P280X145-5N -> TMP006:BGA8DS
- U7: value TMP006 -> BMP180; device TMP006:BGA8DS -> BMP180:BMP180
- U8: value OPA344 -> USD-SOCKETSMD; device OPA344:SOT23-5 -> MicroSD:MICRO-SD-SOCKET-PP
- U9: value ADMP401 -> MIC9.7MM; device ADMP401:ADMP401 -> MIC:MIC-9.7MM
- moved C5 93.2 mm to (15.6, 5.21)
- moved L2 89.3 mm to (27.8, 52.5), flipped to the bottom, turned to 180 degrees
- moved C6 88.1 mm to (14.1, 6.60)
- moved C22 82.8 mm to (8.38, 3.56), turned to 270 degrees
- moved U8 82.1 mm to (20.6, 19.1), flipped to the bottom
- moved C7 80.0 mm to (19.0, 57.4), turned to 90 degrees
- moved C3 78.8 mm to (16.9, 22.6), turned to 90 degrees
- moved R10 78.8 mm to (5.21, 22.6), turned to 270 degrees
- moved L1 77.7 mm to (10.8, -3.30)
- moved R1 74.8 mm to (12.4, 57.1), turned to 90 degrees
- moved R9 74.6 mm to (3.81, 22.6), turned to 270 degrees
- moved C2 74.2 mm to (15.5, 22.6), turned to 270 degrees
- moved C9 72.9 mm to (14.6, -3.30)
- moved R8 72.1 mm to (19.3, 57.3), flipped to the bottom, turned to 270 degrees
- moved R4 71.3 mm to (12.7, 22.6), turned to 90 degrees
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- renumbered LED2 to LED1
Connections:
- removed net BTCX_RF_ACTIVE: U10.9
- removed net BTCX_STATUS: U10.10
- removed net BTCX_TXCONF: U10.11
- removed net BUZZ+: BUZZ.+, U10.41
- removed net BUZZ-: BUZZ.-, U10.40
- removed net PBL: S1.3, U10.43
- removed net PBR: S2.3, U10.44
- removed net RF_SW_CTRL0_ANT0: U10.13
- removed net RF_SW_CTRL3_ANT1: U10.12
- removed net SD_CD: U1.CD, U10.42
- new net BUZZ+/TDO: BUZZ.+, JTAG.7, U1.41
- new net BUZZ-/TCK: BUZZ.-, JTAG.8, U1.40
- new net N$10: C23.2, R14.2, U9.2
- new net PBL/TDI: JTAG.3, S1.3, U1.43
- new net PBR/TMS: JTAG.1, S2.3, U1.44
- new net SD_CD/TRST: JTAG.5, U1.42, U8.CD
- net !MODE: now also S3.2, U1.53; no longer U10.53
- net !RST: now also C22.2, JTAG.6, R13.2, S4.2, U1.26; no longer U10.26
- net +3V3: now also C1.2, C11.1, C12.1, C19.+, C2.2, C20.2, C26.2, C3.1, C4.2, C5.1, CAM.3V3, JTAG.2, LED1.A, R13.1, R14.1, R6.1, R7.2, R8.2, U1.19, U1.20, U1.46, U1.47, U1.49, U10.5, U3.5, U5.VDD, U6.A3, U6.B1, U7.2, U7.3, U8.4; no longer C10.2, C13.2, C19.2, C20.1, C22.1, C24.1, C25.1, C7.2, C8.2, C9.+, LED1.2, R11.2, R13.2, R7.1, SV1.4, U$7.5, U1.4, U10.19, U10.20, U10.46, U10.47, U10.49, U2.2, U2.3, U3.VDD, U7.A3, U7.B1, U8.5, U9.5
- net A0: now also U1.54; no longer U10.54
- net ANT: now also U1.15; no longer U10.15
- net D2: now also U1.3; no longer U10.3
- net ENABLE: now also R2.1, U3.1; no longer R9.1, U$7.1
- net GND: now also C12.2, C19.-, C20.1, C22.1, C26.1, C3.2, C4.1, C8.2, C9.2, CAM.GND, JTAG.4, R1.1, R17.2, S1.2, S2.2, S3.1, S4.1, U1.14, U1.16, U1.17, U1.18, U1.21, U1.29, U1.30, U1.37, U1.45, U1.48, U1.50, U1.55, U1.56, U1.57, U1.58, U1.59, U1.60, U1.61, U1.62, U1.63, U1.64, U1.65, U1.66, U1.67, U10.2, U2.2, U3.2, U5.7, U5.GND, U6.A1, U6.A2, U6.C1, U7.7, U8.6, U8.GND1, U8.GND2, U9.1; no longer C12.1, C19.1, C20.2, C22.2, C23.2, C25.2, C8.1, C9.-, R2.1, R6.2, SV1.1, U$7.2, U1.6, U1.GND1, U1.GND2, U10.14, U10.16, U10.17, U10.18, U10.21, U10.29, U10.30, U10.37, U10.45, U10.48, U10.50, U10.55, U10.56, U10.57, U10.58, U10.59, U10.60, U10.61, U10.62, U10.63, U10.64, U10.65, U10.66, U10.67, U2.7, U3.7, U3.GND, U6.2, U7.A1, U7.A2, U7.C1, U8.2, U9.2, U9.4, U9.6
- net LDR: now also U1.1; no longer U10.1
- net MCU_USB_DM: now also R5.1, U1.52; no longer R8.1, U10.52
- net MCU_USB_DP: now also R4.1, U1.51; no longer R3.1, U10.51
- net MIC: now also C25.1, R18.1, U1.2, U10.1; no longer C4.1, R5.1, U10.2, U8.1
- net MISO: now also U1.25, U8.7; no longer U1.7, U10.25
- net MOSI: now also U1.23, U8.3; no longer U1.3, U10.23
- net N$1: now also C9.1; no longer C11.1
- net N$13: now also R8.1, U6.C2; no longer R13.1, U7.C2
- net N$14: now also C13.2; no longer C12.2
- net N$17: now also R5.2; no longer R8.2
- net N$18: now also R4.2; no longer R3.2
- net N$2: now also C8.1, R2.2, SW.1, U3.4; no longer C3.2, U9.1
- net N$27: now also LED1.G, R10.1; no longer LED1.3, R14.1
- net N$29: now also LED1.B, R11.1; no longer LED1.4, R10.1
- net N$3: now also U3.3; no longer U$7.3
- net N$4: now also R1.2, U2.5; no longer R2.2, U6.5
- net N$5: now also R3.1; no longer R1.1
- net N$54: now also LED1.R, R9.1; no longer LED1.1, R15.1
- net N$6: now also R3.2, U2.1; no longer R1.2, U6.1
- net N$7: now also C23.1, R15.2; no longer C3.1, R4.2
- net N$8: now also C25.2, R15.1, R18.2, U10.4; no longer C4.2, R4.1, R5.2, U8.4
- net N$9: now also C24.1, R16.2, R17.1, U10.3; no longer C5.1, R6.1, R7.2, U8.3
- net RGB_BLUE: now also R11.2, U1.6; no longer R14.2, U10.6
- net RGB_GREEN: now also U1.7; no longer U10.7
- net RGB_RED: now also R9.2, U1.8; no longer R15.2, U10.8
- net RX: now also CAM.RX, U1.38; no longer SV1.3, U10.38
- net SCK: now also U1.24, U8.5; no longer U1.5, U10.24
- net SCL: now also R7.1, U1.5, U5.SCK, U6.B3, U7.5; no longer R11.1, U10.5, U2.5, U3.SCK, U7.B3
- net SDA: now also R6.2, U1.4, U5.DATA, U6.C3, U7.6; no longer R16.2, U10.4, U2.6, U3.DATA, U7.C3
- net SD_CS: now also U1.22, U8.2; no longer U1.2, U10.22
- net TX: now also CAM.TX, U1.39; no longer SV1.2, U10.39
- net UVCC: now also C7.2, U2.4; no longer C1.2, D1.ANODE, U6.4
- net VBAT: now also C10.2, U2.3; no longer C2.2, C23.1, D1.CATHODE, R9.2, SW.1, U$7.4, U10.28, U6.3
- net WKP: now also U1.27; no longer U10.27
Routing:
- net +3V3: track 0.00 -> 55.6 mm, vias 0 -> 9
- net !RST: track 0.00 -> 41.7 mm, vias 0 -> 2
- net N$54: track 0.00 -> 34.2 mm
- net N$29: track 0.00 -> 30.9 mm
- net N$27: track 0.00 -> 29.8 mm
- net PBR/TMS: track 0.00 -> 27.1 mm
- net UVCC: track 0.00 -> 25.1 mm, vias 0 -> 2
- net VBAT: track 0.00 -> 20.2 mm
- net BUZZ-/TCK: track 0.00 -> 20.1 mm
- net BUZZ+/TDO: track 0.00 -> 19.1 mm
- net RGB_RED: track 0.00 -> 13.5 mm
- net PBL/TDI: track 0.00 -> 12.1 mm
- net RGB_GREEN: track 0.00 -> 12.0 mm
- net N$6: track 0.00 -> 11.2 mm
- net SD_CD/TRST: track 0.00 -> 10.6 mm
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- added copper zone on layer 15, net +3V3
- added copper zone on layer 16, net +3V3
- added copper zone on layer 1, net GND
- added copper zone on layer 16, net GND
- added copper zone on layer 2, net GND
- added copper zone on layer 15, net N$11
- added copper zone on layer 2, net N$15
- added copper zone on layer 2, net N$16
- added copper zone on layer 15, net N$19
- added copper zone on layer 16, net N$2
- added copper zone on layer 16, net N$20
- added copper zone on layer 16, net N$21
- added copper zone on layer 15, net N$22
- added copper zone on layer 16, net N$23
- added copper zone on layer 16, net N$3
Other:
- board text added: "Accel"
- board text added: "Gyro"
- board text added: "Mag"
- board text added: "SenSing v3.1 24 FEB 15"
- board text added: "X"
- board text added: "Y"
- board text added: "Z"
